Commit message: Use turtlebot_finger mesh for collision, as current box triggers collisions with the support surface on grasping

File: turtlebot_arm_description/urdf/arm_hardware.xacro (robot description, xacro)
@@ -59,5 +59,5 @@
       <xacro:box_inertia length="0.0783" width="0.03801" height="0.0193" mass="0.015"/>
       <visual>
-        <origin xyz=" 0 0 0 " rpy="0 0 0"/>
+        <origin xyz="0 0 0 " rpy="0 0 0"/>
         <geometry>
           <mesh filename="package://turtlebot_arm_description/meshes/turtlebot_finger.stl" scale="${M_SCALE} ${M_SCALE} ${M_SCALE}"/>
@@ -66,7 +66,7 @@
       </visual>
       <collision>
-        <origin xyz="0.02645 0.0 -0.00655" rpy="0 0 0"/>
-        <geometry>
-          <box size="0.0783 0.03801 0.0193"/>
+        <origin xyz="0 0 0 " rpy="0 0 0"/>
+        <geometry>
+          <mesh filename="package://turtlebot_arm_description/meshes/turtlebot_finger.stl" scale="${M_SCALE} ${M_SCALE} ${M_SCALE}"/>
         </geometry>
       </collision>
@@ -289,6 +289,6 @@
     </gazebo>
   </xacro:macro>
-    <xacro:macro name="pincher_gripper" params="name color *origin">
-      <link name="${name}_link">
+  <xacro:macro name="pincher_gripper" params="name color *origin">
+    <link name="${name}_link">
       <xacro:box_inertia length="0.036" width="0.028" height="0.004" mass="0.00001"/>
       <visual>

Commit message: Set minDepth to 1 mm for fingers to make easier grasping on Gazebo

File: turtlebot_arm_description/urdf/arm_hardware.xacro (robot description, xacro)
@@ -59,5 +59,5 @@
       <xacro:box_inertia length="0.0783" width="0.03801" height="0.0193" mass="0.015"/>
       <visual>
-        <origin xyz="0 0 0 " rpy="0 0 0"/>
+        <origin xyz="0 0 0" rpy="0 0 0"/>
         <geometry>
           <mesh filename="package://turtlebot_arm_description/meshes/turtlebot_finger.stl" scale="${M_SCALE} ${M_SCALE} ${M_SCALE}"/>
@@ -66,5 +66,5 @@
       </visual>
       <collision>
-        <origin xyz="0 0 0 " rpy="0 0 0"/>
+        <origin xyz="0 0 0" rpy="0 0 0"/>
         <geometry>
           <mesh filename="package://turtlebot_arm_description/meshes/turtlebot_finger.stl" scale="${M_SCALE} ${M_SCALE} ${M_SCALE}"/>
@@ -76,4 +76,5 @@
       <selfCollide>true</selfCollide>
       <gravity>true</gravity>
+      <minDepth>0.01</minDepth>
     </gazebo>
   </xacro:macro>
@@ -93,5 +94,5 @@
       </inertial>
       <visual>
-        <origin xyz=" 0 0 0 " rpy="0 0 0"/>
+        <origin xyz="0 0 0" rpy="0 0 0"/>
         <geometry>
           <mesh filename="package://turtlebot_arm_description/meshes/ax12_box.stl" scale="${M_SCALE} ${M_SCALE} ${M_SCALE}"/>
@@ -121,5 +122,5 @@
       <xacro:box_inertia length="0.025" width="0.038" height="0.004" mass="0.004"/>
       <visual>
-        <origin xyz=" 0 0 0 " rpy="0 0 0"/>
+        <origin xyz="0 0 0" rpy="0 0 0"/>
         <geometry>
           <mesh filename="package://turtlebot_arm_description/meshes/F10.stl" scale="${M_SCALE} ${M_SCALE} ${M_SCALE}"/>
@@ -149,5 +150,5 @@
       <xacro:box_inertia length="0.025" width="0.038" height="0.009" mass="0.005"/>
       <visual>
-        <origin xyz=" 0 0 0 " rpy="0 0 0"/>
+        <origin xyz="0 0 0" rpy="0 0 0"/>
         <geometry>
           <mesh filename="package://turtlebot_arm_description/meshes/F3.stl" scale="${M_SCALE} ${M_SCALE} ${M_SCALE}"/>
@@ -180,5 +181,5 @@
       <xacro:box_inertia length="0.025" width="0.038" height="0.009" mass="0.008"/>
       <visual>
-        <origin xyz=" 0 0 0 " rpy="0 0 0"/>
+        <origin xyz="0 0 0" rpy="0 0 0"/>
         <geometry>
           <mesh filename="package://turtlebot_arm_description/meshes/F3.stl" scale="${M_SCALE} ${M_SCALE} ${M_SCALE}"/>
@@ -211,5 +212,5 @@
       <xacro:box_inertia length="0.025" width="0.0485" height="0.0375" mass="0.010"/>
       <visual>
-        <origin xyz=" 0 0 0 " rpy="0 0 0"/>
+        <origin xyz="0 0 0" rpy="0 0 0"/>
         <geometry>
           <mesh filename="package://turtlebot_arm_description/meshes/F2.stl" scale="${M_SCALE} ${M_SCALE} ${M_SCALE}"/>
@@ -242,5 +243,5 @@
       <xacro:box_inertia length="0.028" width="0.0485" height="0.065" mass="0.016"/>
       <visual>
-        <origin xyz=" 0 0 0 " rpy="0 0 0"/>
+        <origin xyz="0 0 0" rpy="0 0 0"/>
         <geometry>
           <mesh filename="package://turtlebot_arm_description/meshes/F4.stl" scale="${M_SCALE} ${M_SCALE} ${M_SCALE}"/>

Commit message: Fix box_inertia macro and use it everywhere

File: turtlebot_arm_description/urdf/arm_hardware.xacro (robot description, xacro)
@@ -4,20 +4,20 @@
   <xacro:property name="M_PI" value="3.14159"/>
   <xacro:property name="M_SCALE" value="0.001"/>
+  <xacro:property name="F2_HEIGHT" value="0.0265"/>
+  <xacro:property name="F3_HEIGHT" value="0.009"/>
+  <xacro:property name="F4_HEIGHT" value="0.0525"/>
   <xacro:property name="F10_HEIGHT" value="0.004"/>
-  <xacro:property name="F4_HEIGHT" value="0.0525"/>
-  <xacro:property name="F3_HEIGHT" value="0.009"/>
   <xacro:property name="AX12_HEIGHT" value="0.0385"/>
   <xacro:property name="AX12_WIDTH" value="0.038"/>
   <xacro:property name="AX12_LENGTH" value="0.050"/>
-  <xacro:property name="F2_HEIGHT" value="0.0265"/>
   <!-- Calculates the inertial properties of a bounding box. From
        https://en.wikipedia.org/wiki/List_of_moments_of_inertia#List_of_3D_inertia_tensors-->
-  <xacro:macro name="box_inertia" params="length width height mass">
+  <xacro:macro name="box_inertia" params="length width height mass x=0 y=0 z=0">
     <inertial>
       <mass value="${mass}"/>
-      <origin xyz="0 0 0"/>
-      <inertia ixx="${mass/12*(height**2+length**2)}" ixy="0" ixz = "0"
-               iyy="${mass/12*(width**2+length**2)}" iyz="0"
-               izz="${mass/12*(width**2+height**2)}"/>
+      <origin xyz="${x} ${y} ${z}"/>
+      <inertia ixx="${mass/12*(width**2+height**2)}" ixy="0" ixz="0"
+               iyy="${mass/12*(length**2+height**2)}" iyz="0"
+               izz="${mass/12*(width**2+length**2)}"/>
     </inertial>
   </xacro:macro>
@@ -86,11 +86,5 @@
     </joint>
     <link name="${name}_link">
-      <inertial>
-        <mass value="0.055"/>
-        <origin xyz="0 0 0"/>
-        <inertia ixx="0.000017012" ixy="0.0" ixz="0.0"
-                 iyy="0.000013258" iyz="0.0"
-                 izz="0.000009483"/>
-      </inertial>
+      <xacro:box_inertia length="${AX12_HEIGHT}" width="${AX12_WIDTH}" height="${AX12_LENGTH}" mass="0.055" z="-0.01241"/>
       <visual>
         <origin xyz="0 0 0" rpy="0 0 0"/>
@@ -103,5 +97,5 @@
         <origin xyz="0.0 0.0 -0.01241" rpy="0 0 0"/>
         <geometry>
-          <box size="0.025 0.038 0.04762"/>
+          <box size="${AX12_HEIGHT} ${AX12_WIDTH} ${AX12_LENGTH}"/>
         </geometry>
       </collision>

File: turtlebot_arm_description/urdf/turtlebot_gripper.xacro (robot description, xacro)
@@ -18,11 +18,5 @@
     </joint>
     <link name="gripper_active_link">
-      <inertial>
-        <mass value="0.010"/>
-        <origin xyz="0 0 0"/>
-        <inertia ixx="0.000001" ixy="0.0" ixz="0.0"
-                 iyy="0.000001" iyz="0.0"
-                 izz="0.000001"/>
-      </inertial>
+      <xacro:box_inertia length="0.025" width="0.0485" height="0.0375" mass="0.010"/>
       <visual>
         <origin xyz=" 0 0 0 " rpy="0 0 0"/>
@@ -56,5 +50,5 @@
       <xacro:box_inertia length="0.025" width="0.038" height="0.009" mass="0.005"/>
       <visual>
-        <origin xyz="0 0 0 " rpy="0 0 0"/>
+        <origin xyz="0 0 0" rpy="0 0 0"/>
         <geometry>
           <mesh filename="package://turtlebot_arm_description/meshes/F3.stl" scale="${M_SCALE} ${M_SCALE} ${M_SCALE}"/>

Commit message: Add AX12_RANGE property: AX-12 servo operational angle (300 degrees)

File: turtlebot_arm_description/urdf/arm_hardware.xacro (robot description, xacro)
@@ -11,4 +11,5 @@
   <xacro:property name="AX12_WIDTH" value="0.038"/>
   <xacro:property name="AX12_LENGTH" value="0.050"/>
+  <xacro:property name="AX12_RANGE" value="5.236"/>  <!-- 300 degrees -->
   <!-- Calculates the inertial properties of a bounding box. From
        https://en.wikipedia.org/wiki/List_of_moments_of_inertia#List_of_3D_inertia_tensors-->
