Commit message: Displace gripper link within the gripper paddles to easy grasping

File: turtlebot_arm_description/urdf/turtlebot_arm.urdf (robot description, URDF)
Before this commit: robot turtlebot_arm, 25 links, 24 joints
Links:
- link arm_elbow_flex_servo_link: geometry collision box size=0.0385 0.038 0.05; visual mesh filename=package://turtlebot_arm_description/meshes/ax12_box.stl scale=0.001 0.001 0.001
- link arm_shoulder_lift_servo_link: geometry collision box size=0.0385 0.038 0.05; visual mesh filename=package://turtlebot_arm_description/meshes/ax12_box.stl scale=0.001 0.001 0.001
- link arm_shoulder_pan_servo_link: geometry collision box size=0.0385 0.038 0.05; visual mesh filename=package://turtlebot_arm_description/meshes/ax12_box.stl scale=0.001 0.001 0.001
- link arm_wrist_flex_servo_link: geometry collision box size=0.0385 0.038 0.05; visual mesh filename=package://turtlebot_arm_description/meshes/ax12_box.stl scale=0.001 0.001 0.001
- link gripper_active_finger_link: geometry collision mesh filename=package://turtlebot_arm_description/meshes/turtlebot_finger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 scale=0.001 0.001 0.001; visual mesh filename=package://turtlebot_arm_description/meshes/turtlebot_finger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 scale=0.001 0.001 0.001
- link gripper_active_link: mass 0.010 -> 0.01
- link gripper_servo_link: geometry collision box size=0.0385 0.038 0.05; visual mesh filename=package://turtlebot_arm_description/meshes/ax12_box.stl scale=0.001 0.001 0.001
- link gripper_static_finger_link: geometry collision mesh filename=package://turtlebot_arm_description/meshes/turtlebot_finger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 scale=0.001 0.001 0.001; visual mesh filename=package://turtlebot_arm_description/meshes/turtlebot_finger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 scale=0.001 0.001 0.001
Joints:
- joint gripper_link_joint: limit lower=-3.14 upper=3.14 effort=30 velocity=1 -> lower=-3.14159 upper=3.14159 effort=30 velocity=1; origin xyz=0 0 0.112 rpy=0 -1.57 0 -> xyz=0 0 0.1 rpy=0 -1.570795 0
- joint gripper_static_joint: axis (none) -> 0 1 0; limit (none) -> lower=0.0 upper=0.0 effort=30 velocity=0.0; type fixed -> revolute

File: turtlebot_arm_description/urdf/turtlebot_arm.xacro (robot description, xacro)
@@ -27,8 +27,8 @@
     <link name="gripper_link"/>
     <joint name="gripper_link_joint" type="revolute">
-      <origin xyz="0 0 0.112" rpy="0 -1.57 0"/>
+      <origin xyz="0 0 0.1" rpy="0 ${-M_PI/2} 0"/>
       <parent link="arm_wrist_flex_link"/>
       <child link="gripper_link"/>
-      <limit effort="30" velocity="1" lower="-3.14" upper="3.14"/>
+      <limit effort="30" velocity="1" lower="${-M_PI}" upper="${M_PI}"/>
       <axis xyz="1 0 0"/>
     </joint>
